File: esp32_light_switch.kicad_sch (KiCad schematic)
At the start: 26 parts, among them J1 Conn_USART0, J2 Screw_Terminal_01x02, J3 Conn_01x02, K1 G5LE-1, Q1 MMBT2222A, SW1 SW_SPST, SW2 SW_SPST, U1 ESP32-WROOM-32E, U2 PC817, U3 MIC5205-3.0YM5

Commit message: refactor to use TRIAC and draw initial pcb
Parts:
- removed D1: D, Diode_SMD:D_SMA_Handsoldering, symbol Device:D
- removed K1: G5LE-1, Relay_THT:Relay_SPDT_Omron-G5LE-1, symbol Relay:G5LE-1
- removed Q1: MMBT2222A, Package_TO_SOT_SMD:SOT-23, symbol Transistor_BJT:MMBT2222A
- added C9: 0.1uF, Capacitor_SMD:C_0805_2012Metric_Pad1.18x1.45mm_HandSolder, symbol Device:C
- added D1: WS2812B, LED_SMD:LED_WS2812B_PLCC4_5.0x5.0mm_P3.2mm, symbol LED:WS2812B
- added Q2: BTB16-800B, Package_TO_SOT_THT:TO-220-3_Vertical, symbol Triac_Thyristor:BTB16-800B
- added R5, R6: 100, Resistor_SMD:R_0805_2012Metric_Pad1.20x1.40mm_HandSolder, symbol Device:R
- J1: footprint Connector_PinHeader_2.54mm:PinHeader_1x02_P2.54mm_Horizontal -> Connector_PinHeader_2.54mm:PinHeader_1x02_P2.54mm_Vertical
- J3: footprint Button_Switch_THT:Toggle BTN -> Connector_PinHeader_2.54mm:PinHeader_1x02_P2.54mm_Vertical
Connections:
- net 220VL: now also U2.4, Q2.2 (A2)
- net 220VN: now also Q2.1 (A1)
- net 3V3: now also C9.1, D1.1 (VDD)
- net 5V: no longer U2.4
- net GND: now also C9.2, D1.3 (VSS)
- net at U2.3: now also R5.1
- net LED_CTRL: now reaches U1.10 (IO25)
- net LED_CTRL: now also R6.1
- new net: Q2.3 (G), R5.2
- new net: D1.4 (DIN), R6.2
Other:
- note added: "LED Control"
- note added: "TRIAC Control"
- note removed: "Relay Control"
- moved on the sheet: C8, J3, R3
